File: resources/camera_board/camera_board.sch (KiCad schematic (older format))
At the start: 10 parts, among them P1 CONN_01X02

Commit message: added new pcb version of camera board for wired leds
Parts:
- D1, D2, D3, D4, D5, D6, D7, D8: footprint custom:LED_SMD_5050 -> LEDs:LED-3MM
- RP1: footprint Housings_DIP:DIP-18_W7.62mm -> Housings_DIP:DIP-16_W7.62mm
Changed lines of the file:
@@
 F 0 "D1" H 3750 3950 50  0000 C CNN
 F 1 "LED" H 3750 3750 50  0000 C CNN
-F 2 "custom:LED_SMD_5050" H 3750 3850 50  0001 C CNN
+F 2 "LEDs:LED-3MM" H 3750 3850 50  0001 C CNN
 F 3 "" H 3750 3850 50  0000 C CNN
 	1    3750 3850
@@
 F 0 "D2" H 4050 3950 50  0000 C CNN
 F 1 "LED" H 4050 3750 50  0000 C CNN
-F 2 "custom:LED_SMD_5050" H 4050 3850 50  0001 C CNN
+F 2 "LEDs:LED-3MM" H 4050 3850 50  0001 C CNN
 F 3 "" H 4050 3850 50  0000 C CNN
 	1    4050 3850
@@
 F 0 "D3" H 4350 3950 50  0000 C CNN
 F 1 "LED" H 4350 3750 50  0000 C CNN
-F 2 "custom:LED_SMD_5050" H 4350 3850 50  0001 C CNN
+F 2 "LEDs:LED-3MM" H 4350 3850 50  0001 C CNN
 F 3 "" H 4350 3850 50  0000 C CNN
 	1    4350 3850
@@
 F 0 "D4" H 4650 3950 50  0000 C CNN
 F 1 "LED" H 4650 3750 50  0000 C CNN
-F 2 "custom:LED_SMD_5050" H 4650 3850 50  0001 C CNN
+F 2 "LEDs:LED-3MM" H 4650 3850 50  0001 C CNN
 F 3 "" H 4650 3850 50  0000 C CNN
 	1    4650 3850
@@
 F 0 "D5" H 4950 3950 50  0000 C CNN
 F 1 "LED" H 4950 3750 50  0000 C CNN
-F 2 "custom:LED_SMD_5050" H 4950 3850 50  0001 C CNN
+F 2 "LEDs:LED-3MM" H 4950 3850 50  0001 C CNN
 F 3 "" H 4950 3850 50  0000 C CNN
 	1    4950 3850
@@
 F 0 "D6" H 5250 3950 50  0000 C CNN
 F 1 "LED" H 5250 3750 50  0000 C CNN
-F 2 "custom:LED_SMD_5050" H 5250 3850 50  0001 C CNN
+F 2 "LEDs:LED-3MM" H 5250 3850 50  0001 C CNN
 F 3 "" H 5250 3850 50  0000 C CNN
 	1    5250 3850
@@
 F 0 "D7" H 5550 3950 50  0000 C CNN
 F 1 "LED" H 5550 3750 50  0000 C CNN
-F 2 "custom:LED_SMD_5050" H 5550 3850 50  0001 C CNN
+F 2 "LEDs:LED-3MM" H 5550 3850 50  0001 C CNN
 F 3 "" H 5550 3850 50  0000 C CNN
 	1    5550 3850
@@
 F 0 "D8" H 5850 3950 50  0000 C CNN
 F 1 "LED" H 5850 3750 50  0000 C CNN
-F 2 "custom:LED_SMD_5050" H 5850 3850 50  0001 C CNN
+F 2 "LEDs:LED-3MM" H 5850 3850 50  0001 C CNN
 F 3 "" H 5850 3850 50  0000 C CNN
 	1    5850 3850
@@
 F 0 "RP1" H 4800 3300 50  0000 C CNN
 F 1 "R_PACK8" H 4800 2400 50  0000 C CNN
-F 2 "Housings_DIP:DIP-18_W7.62mm" H 4800 2850 50  0001 C CNN
+F 2 "Housings_DIP:DIP-16_W7.62mm" H 4800 2850 50  0001 C CNN
 F 3 "" H 4800 2850 50  0000 C CNN
 	1    4800 2850
