File: resources/camera_board_v1.1/camera_board.sch (KiCad schematic (older format))
At the start: 10 parts, among them P1 CONN_01X02

Commit message: changed pcb layout, changed installation instructions
Parts:
- P1: footprint Socket_Strips:Socket_Strip_Straight_1x02 -> Pin_Headers:Pin_Header_Angled_1x02
Changed lines of the file:
@@
 F 0 "P1" H 3100 2350 50  0000 C CNN
 F 1 "CONN_01X02" V 3200 2200 50  0000 C CNN
-F 2 "Socket_Strips:Socket_Strip_Straight_1x02" H 3100 2200 50  0001 C CNN
+F 2 "Pin_Headers:Pin_Header_Angled_1x02" H 3100 2200 50  0001 C CNN
 F 3 "" H 3100 2200 50  0000 C CNN
 	1    3100 2200
