File: resources/hardware/camera_board_smd/camera_board.sch (KiCad schematic (older format))
At the start: 10 parts, among them P1 CONN_01X02

Commit message: new designs for pcbs
Parts:
- removed D5, D6, D7, D8: LED_RGB, custom:SMD-LED_5250, symbol LED_RGB
- removed P1: CONN_01X02, Pin_Headers:Pin_Header_Angled_2x01, symbol CONN_01X02
- removed RP1: R_PACK8, Housings_DIP:DIP-16_W7.62mm, symbol R_PACK8
- added P1: CONN_01X03, Pin_Headers:Pin_Header_Angled_1x03, symbol CONN_01X03
- added Q1: Q_NPN_EBC, TO_SOT_Packages_THT:TO-92_Inline_Wide, symbol Q_NPN_EBC
- added R1, R2, R3, R4, R5: R_Small, Resistors_ThroughHole:Resistor_Horizontal_RM10mm, symbol R_Small
Connections:
- net labels added: SGNL
- wire segments 58 -> 10
