File: resources/hardware/camera_board/camera_board.sch (KiCad schematic (older format))
At the start: 11 parts, among them P1 CONN_01X03, Q1 Q_NPN_EBC

Commit message: added letterbox-setup.py
Parts:
- R1, R2, R3, R4: value R_Small -> 33 Ohm
- R5: value R_Small -> 330 Ohm
Changed lines of the file:
@@
 P 3950 3400
 F 0 "R1" H 3980 3420 50  0000 L CNN
-F 1 "R_Small" H 3980 3360 50  0000 L CNN
+F 1 "33 Ohm" H 3980 3360 50  0000 L CNN
 F 2 "Resistors_ThroughHole:Resistor_Horizontal_RM10mm" H 3950 3400 50  0001 C CNN
 F 3 "" H 3950 3400 50  0000 C CNN
@@
 P 4750 3400
 F 0 "R2" H 4780 3420 50  0000 L CNN
-F 1 "R_Small" H 4780 3360 50  0000 L CNN
+F 1 "33 Ohm" H 4780 3360 50  0000 L CNN
 F 2 "Resistors_ThroughHole:Resistor_Horizontal_RM10mm" H 4750 3400 50  0001 C CNN
 F 3 "" H 4750 3400 50  0000 C CNN
@@
 P 5550 3400
 F 0 "R3" H 5580 3420 50  0000 L CNN
-F 1 "R_Small" H 5580 3360 50  0000 L CNN
+F 1 "33 Ohm" H 5580 3360 50  0000 L CNN
 F 2 "Resistors_ThroughHole:Resistor_Horizontal_RM10mm" H 5550 3400 50  0001 C CNN
 F 3 "" H 5550 3400 50  0000 C CNN
@@
 P 6350 3400
 F 0 "R4" H 6380 3420 50  0000 L CNN
-F 1 "R_Small" H 6380 3360 50  0000 L CNN
+F 1 "33 Ohm" H 6380 3360 50  0000 L CNN
 F 2 "Resistors_ThroughHole:Resistor_Horizontal_RM10mm" H 6350 3400 50  0001 C CNN
 F 3 "" H 6350 3400 50  0000 C CNN
@@
 P 3350 4200
 F 0 "R5" H 3380 4220 50  0000 L CNN
-F 1 "R_Small" H 3380 4160 50  0000 L CNN
+F 1 "330 Ohm" H 3380 4160 50  0000 L CNN
 F 2 "Resistors_ThroughHole:Resistor_Horizontal_RM10mm" H 3350 4200 50  0001 C CNN
 F 3 "" H 3350 4200 50  0000 C CNN
