File: resources/hardware/head_board/head_board.sch (KiCad schematic (older format))
At the start: 18 parts, among them IC1 ATMEGA328P-P, P1 SERIAL/RST, P2 PI_CONN, P3 REED, P4 PR, P5 CAM_LEDS, P6 STEPPER, P7 PR_LED, P8 FDBK_LED, U1 ULN2003

Commit message: added letterbox-setup.py
Parts:
- C1: value CP1 -> 10 uF
- R1: value R -> 56 Ohm
- R2: value R -> 10 kOhm
- R5, R6: value R -> 100 Ohm
Connections:
- net PIRX: now also IC1.3 ((PCINT17/TXD)PD1), P1.3 (P3); no longer IC1.2 ((PCINT16/RXD)PD0), P1.2 (P2)
- net PITX: now also IC1.2 ((PCINT16/RXD)PD0), P1.2 (P2); no longer IC1.3 ((PCINT17/TXD)PD1), P1.3 (P3)
- net RST: now also R2.2
- net at C1.2, P1.1 (P1): no longer R2.2
Other:
- moved on the sheet: C1, P1, R2
Changed lines of the file:
@@
 L CONN_01X03 P1
 U 1 1 56E6F37A
-P 5400 5800
-F 0 "P1" H 5400 6000 50  0000 C CNN
-F 1 "SERIAL/RST" V 5500 5800 50  0000 C CNN
-F 2 "Pin_Headers:Pin_Header_Straight_1x03" H 5400 5800 50  0001 C CNN
-F 3 "" H 5400 5800 50  0000 C CNN
-	1    5400 5800
+P 5400 6050
+F 0 "P1" H 5400 6250 50  0000 C CNN
+F 1 "SERIAL/RST" V 5500 6050 50  0000 C CNN
+F 2 "Pin_Headers:Pin_Header_Straight_1x03" H 5400 6050 50  0001 C CNN
+F 3 "" H 5400 6050 50  0000 C CNN
+	1    5400 6050
 	0    1    1    0
 $EndComp
@@
 Wire Wire Line
 	6150 4350 6550 4350
+Text Label 4800 4150 0    60   ~ 0
+PIRX
 Text Label 4800 4050 0    60   ~ 0
-PIRX
-Text Label 4800 4150 0    60   ~ 0
 PITX
 Wire Wire Line
@@
 P 8450 2950
 F 0 "R5" V 8530 2950 50  0000 C CNN
-F 1 "R" V 8450 2950 50  0000 C CNN
+F 1 "100 Ohm" V 8450 2950 50  0000 C CNN
 F 2 "Resistors_ThroughHole:Resistor_Horizontal_RM7mm" V 8380 2950 50  0001 C CNN
 F 3 "" H 8450 2950 50  0000 C CNN
@@
 P 8950 4850
 F 0 "R6" V 9030 4850 50  0000 C CNN
-F 1 "R" V 8950 4850 50  0000 C CNN
+F 1 "100 Ohm" V 8950 4850 50  0000 C CNN
 F 2 "Resistors_ThroughHole:Resistor_Horizontal_RM7mm" V 8880 4850 50  0001 C CNN
 F 3 "" H 8950 4850 50  0000 C CNN
@@
 $EndComp
 Wire Wire Line
-	5300 4150 5300 5600
-Wire Wire Line
-	5400 4050 5400 5600
+	5300 4150 5300 5850
+Wire Wire Line
+	5400 4050 5400 5850
 $Comp
 L CP1 C1
 U 1 1 56E7E788
-P 5600 5300
-F 0 "C1" H 5625 5400 50  0000 L CNN
-F 1 "CP1" H 5625 5200 50  0000 L CNN
-F 2 "Capacitors_ThroughHole:C_Radial_D5_L11_P2" H 5600 5300 50  0001 C CNN
-F 3 "" H 5600 5300 50  0000 C CNN
-	1    5600 5300
+P 5600 5700
+F 0 "C1" H 5625 5800 50  0000 L CNN
+F 1 "10 uF" H 5625 5600 50  0000 L CNN
+F 2 "Capacitors_ThroughHole:C_Radial_D5_L11_P2" H 5600 5700 50  0001 C CNN
+F 3 "" H 5600 5700 50  0000 C CNN
+	1    5600 5700
 	1    0    0    -1
 $EndComp
 Wire Wire Line
-	5500 5600 5800 5600
-Wire Wire Line
-	5600 5600 5600 5450
-Wire Wire Line
-	5600 5150 5600 3900
+	5600 5550 5800 5550
+Wire Wire Line
+	5600 3900 5600 5550
 Wire Wire Line
 	5600 3900 4800 3900
-Connection ~ 5600 5600
 $Comp
 L R R2
 U 1 1 56E7E8E4
-P 5950 5600
-F 0 "R2" V 6030 5600 50  0000 C CNN
-F 1 "R" V 5950 5600 50  0000 C CNN
-F 2 "Resistors_ThroughHole:Resistor_Horizontal_RM7mm" V 5880 5600 50  0001 C CNN
-F 3 "" H 5950 5600 50  0000 C CNN
-	1    5950 5600
+P 5950 5550
+F 0 "R2" V 6030 5550 50  0000 C CNN
+F 1 "10 kOhm" V 5950 5550 50  0000 C CNN
+F 2 "Resistors_ThroughHole:Resistor_Horizontal_RM7mm" V 5880 5550 50  0001 C CNN
+F 3 "" H 5950 5550 50  0000 C CNN
+	1    5950 5550
 	0    1    1    0
 $EndComp
@@
 L +3.3V #PWR018
 U 1 1 56E7E98E
-P 6100 5600
-F 0 "#PWR018" H 6100 5450 50  0001 C CNN
-F 1 "+3.3V" H 6100 5740 50  0000 C CNN
-F 2 "" H 6100 5600 50  0000 C CNN
-F 3 "" H 6100 5600 50  0000 C CNN
-	1    6100 5600
+P 6100 5550
+F 0 "#PWR018" H 6100 5400 50  0001 C CNN
+F 1 "+3.3V" H 6100 5690 50  0000 C CNN
+F 2 "" H 6100 5550 50  0000 C CNN
+F 3 "" H 6100 5550 50  0000 C CNN
+	1    6100 5550
 	0    1    1    0
 $EndComp
@@
 P 5550 2950
 F 0 "R1" V 5630 2950 50  0000 C CNN
-F 1 "R" V 5550 2950 50  0000 C CNN
+F 1 "56 Ohm" V 5550 2950 50  0000 C CNN
 F 2 "Resistors_ThroughHole:Resistor_Horizontal_RM7mm" V 5480 2950 50  0001 C CNN
 F 3 "" H 5550 2950 50  0000 C CNN
@@
 Wire Wire Line
 	6050 4250 6350 4250
+Wire Wire Line
+	5500 5850 5600 5850
 $EndSCHEMATC
