File: resources/hardware/head_board/head_board.sch (KiCad schematic (older format))
At the start: 23 parts, among them IC1 ATMEGA328P-P, P1 SERIAL, P2 PI_CONN, P3 REED, P4 PR, P5 CAM_LEDS, P6 STEPPER, P7 PR_LED, P8 FDBK_LED, Q1 BC547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

Commit message: finished new headboard pcbs
Connections:
- net +3V3: no longer P2.17 (P17)
- net FDBK: now also P2.31 (P31); no longer P2.18 (P18)
- no-connect marks 38 -> 39
Other:
- moved on the sheet: P5

Commit message: fixed some pcbs issues
Connections:
- net PIRX: now also P1.5 (P5); no longer P1.4 (P4)
- net PITX: now also P1.4 (P4); no longer P1.5 (P5)
Changed lines of the file:
@@
 	6550 2450 6550 4250
 Wire Wire Line
-	4750 1350 4950 1350
-Wire Wire Line
-	4950 1350 5050 1350
+	4750 1350 5050 1350
 Wire Wire Line
 	5250 1350 5250 1050
@@
 	9100 4050 9100 3200
 Wire Wire Line
-	5300 4150 5300 6100
+	5300 4150 5300 6600
 Wire Wire Line
 	5400 4050 5400 6300
@@
 	5650 6600 5700 6600
 Wire Wire Line
-	5450 6800 5450 6650
-Wire Wire Line
-	5450 6650 5300 6650
-Wire Wire Line
-	5300 6650 5300 6300
-Wire Wire Line
 	5750 6800 5750 6650
 Wire Wire Line
@@
 	5150 5850 5150 6800
 Wire Wire Line
-	5500 6600 5500 6100
-Wire Wire Line
 	5700 6600 5700 6400
-Wire Wire Line
-	5500 6100 5300 6100
-Wire Wire Line
-	5300 6300 5400 6300
 Wire Wire Line
 	4950 1850 4950 1950
@@
 	1    0    0    -1
 $EndComp
+Wire Wire Line
+	5300 6600 5450 6600
+Wire Wire Line
+	5450 6600 5450 6800
+Wire Wire Line
+	5500 6600 5500 6300
+Wire Wire Line
+	5500 6300 5400 6300
 $EndSCHEMATC
