File: resources/hardware/head_board/head_board.kicad_pcb (KiCad board)
At the start: 2 copper layers, 66 x 61 mm, 23 parts, among them IC1 ATMEGA328P-P, P1 SERIAL, P2 PI_CONN, P3 REED, P4 PR, P5 CAM_LEDS, P6 STEPPER, P7 PR_LED, P8 FDBK_LED, Q1 BC547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

Commit message: fixed some pcbs issues
Connections:
- P1 pad 4: /PIRX -> /PITX
- P1 pad 5: /PITX -> /PIRX
Routing:
- net /PITX: track 140.8 -> 146.0 mm, vias 1 -> 3
- net /PIRX: track 138.6 -> 140.9 mm
Other:
- board text added: "CAM"
- board text added: "LED"
- board text added: "R"
- board text added: "STP"
- board text added: "T"
- board text removed: "RX"
- board text removed: "TX"
Changed lines of the file:
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@@
     (links 56)
     (no_connects 6)
-    (area 124.25646 98.374999 191.075001 160.465)
+    (area 124.924999 98.374999 191.075001 159.575001)
     (thickness 1.6)
-    (drawings 28)
-    (tracks 217)
+    (drawings 32)
+    (tracks 228)
     (zones 0)
     (modules 23)
@@
       (net 7 +3V3))
     (pad 4 thru_hole oval (at 0 7.62) (size 2.032 1.7272) (drill 1.016) (layers *.Cu *.Mask F.SilkS)
+      (net 5 /PITX))
+    (pad 5 thru_hole oval (at 0 10.16) (size 2.032 1.7272) (drill 1.016) (layers *.Cu *.Mask F.SilkS)
       (net 4 /PIRX))
-    (pad 5 thru_hole oval (at 0 10.16) (size 2.032 1.7272) (drill 1.016) (layers *.Cu *.Mask F.SilkS)
-      (net 5 /PITX))
     (pad 6 thru_hole oval (at 0 12.7) (size 2.032 1.7272) (drill 1.016) (layers *.Cu *.Mask F.SilkS)
       (net 24 /DTR))
@@
       (net 23 "Net-(Q2-Pad2)"))
   )
-  (gr_text + (at 153 145.25) (layer F.Cu)
+  (gr_text LED (at 129.25 127.25 90) (layer F.Cu)
+    (effects (font (size 1.5 1.5) (thickness 0.3)))
+  )
+  (gr_text CAM (at 135.5 117.25 90) (layer F.Cu)
+    (effects (font (size 1.5 1.5) (thickness 0.3)))
+  )
+  (gr_text STP (at 151.75 113.25) (layer F.Cu)
+    (effects (font (size 1.5 1.5) (thickness 0.3)))
+  )
+  (gr_text + (at 148.25 115.25) (layer F.Cu)
+    (effects (font (size 1.5 1.5) (thickness 0.3)))
+  )
+  (gr_text + (at 153 144.5) (layer F.Cu)
     (effects (font (size 1.5 1.5) (thickness 0.3)))
   )
@@
     (effects (font (size 1.5 1.5) (thickness 0.3)))
   )
-  (gr_text TX (at 152.5 148) (layer F.Cu)
+  (gr_text T (at 159 148.25) (layer F.Cu)
     (effects (font (size 1.5 1.5) (thickness 0.3)))
   )
@@
     (effects (font (size 1.5 1.5) (thickness 0.3)))
   )
-  (gr_text RX (at 152.5 150.5) (layer F.Cu)
+  (gr_text R (at 153 150.5) (layer F.Cu)
     (effects (font (size 1.5 1.5) (thickness 0.3)))
   )
@@
   (segment (start 135.128 125.476) (end 135.636 125.984) (width 0.8) (layer B.Cu) (net 3))
   (segment (start 133.096 125.476) (end 135.128 125.476) (width 0.8) (layer B.Cu) (net 3))
-  (segment (start 162.56 136.144) (end 162.56 134.112) (width 0.8) (layer B.Cu) (net 4))
-  (segment (start 161.544 147.828) (end 162.56 146.812) (width 0.8) (layer B.Cu) (net 4))
-  (segment (start 155.956 147.828) (end 161.544 147.828) (width 0.8) (layer B.Cu) (net 4))
-  (segment (start 162.56 136.144) (end 162.56 146.812) (width 0.8) (layer B.Cu) (net 4))
-  (segment (start 163.576 133.096) (end 168.656 133.096) (width 0.8) (layer F.Cu) (net 4))
-  (segment (start 163.068 133.604) (end 163.576 133.096) (width 0.8) (layer F.Cu) (net 4))
-  (via (at 163.068 133.604) (size 1.7) (drill 0.8) (layers F.Cu B.Cu) (net 4))
-  (segment (start 162.56 134.112) (end 163.068 133.604) (width 0.8) (layer B.Cu) (net 4))
-  (segment (start 143.66 101.704) (end 143.66 105.16) (width 0.8) (layer F.Cu) (net 4))
-  (segment (start 168.656 133.096) (end 186.944 133.096) (width 0.8) (layer F.Cu) (net 4))
-  (segment (start 186.944 133.096) (end 188.976 131.064) (width 0.8) (layer F.Cu) (net 4))
-  (segment (start 188.976 131.064) (end 188.976 102.616) (width 0.8) (layer F.Cu) (net 4))
-  (segment (start 188.976 102.616) (end 186.436 100.076) (width 0.8) (layer F.Cu) (net 4))
-  (segment (start 186.436 100.076) (end 145.288 100.076) (width 0.8) (layer F.Cu) (net 4))
-  (segment (start 145.288 100.076) (end 143.66 101.704) (width 0.8) (layer F.Cu) (net 4))
-  (segment (start 166.624 133.096) (end 168.656 133.096) (width 0.8) (layer F.Cu) (net 4))
-  (segment (start 146.05 148.59) (end 148.082 148.59) (width 0.8) (layer B.Cu) (net 4))
-  (segment (start 148.844 147.828) (end 155.956 147.828) (width 0.8) (layer B.Cu) (net 4))
-  (segment (start 148.082 148.59) (end 148.844 147.828) (width 0.8) (layer B.Cu) (net 4))
-  (segment (start 164.592 141.732) (end 164.592 135.128) (width 0.8) (layer B.Cu) (net 5))
-  (segment (start 163.068 150.368) (end 164.592 148.844) (width 0.8) (layer B.Cu) (net 5))
-  (segment (start 164.592 148.844) (end 164.592 141.732) (width 0.8) (layer B.Cu) (net 5))
-  (segment (start 155.956 150.368) (end 163.068 150.368) (width 0.8) (layer B.Cu) (net 5))
-  (segment (start 141.12 101.704) (end 141.12 105.16) (width 0.8) (layer F.Cu) (net 5))
-  (segment (start 141.224 101.6) (end 141.12 101.704) (width 0.8) (layer F.Cu) (net 5))
-  (via (at 141.224 101.6) (size 1.7) (drill 0.8) (layers F.Cu B.Cu) (net 5))
-  (segment (start 142.748 100.076) (end 141.224 101.6) (width 0.8) (layer B.Cu) (net 5))
-  (segment (start 186.436 100.076) (end 142.748 100.076) (width 0.8) (layer B.Cu) (net 5))
-  (segment (start 188.976 102.616) (end 186.436 100.076) (width 0.8) (layer B.Cu) (net 5))
-  (segment (start 188.976 131.064) (end 188.976 102.616) (width 0.8) (layer B.Cu) (net 5))
-  (segment (start 186.944 133.096) (end 188.976 131.064) (width 0.8) (layer B.Cu) (net 5))
-  (segment (start 166.624 133.096) (end 186.944 133.096) (width 0.8) (layer B.Cu) (net 5))
-  (segment (start 164.592 135.128) (end 166.624 133.096) (width 0.8) (layer B.Cu) (net 5))
-  (segment (start 146.05 151.13) (end 148.082 151.13) (width 0.8) (layer B.Cu) (net 5))
-  (segment (start 148.844 150.368) (end 155.956 150.368) (width 0.8) (layer B.Cu) (net 5))
-  (segment (start 148.082 151.13) (end 148.844 150.368) (width 0.8) (layer B.Cu) (net 5))
+  (segment (start 164.592 142) (end 164.592 137.092) (width 0.8) (layer B.Cu) (net 4))
+  (segment (start 143.66 102.34) (end 143.66 105.16) (width 0.8) (layer F.Cu) (net 4))
+  (segment (start 146 100) (end 143.66 102.34) (width 0.8) (layer F.Cu) (net 4))
+  (segment (start 187.25 100) (end 146 100) (width 0.8) (layer F.Cu) (net 4))
+  (segment (start 189.5 102.25) (end 187.25 100) (width 0.8) (layer F.Cu) (net 4))
+  (segment (start 189.5 129.75) (end 189.5 102.25) (width 0.8) (layer F.Cu) (net 4))
+  (segment (start 187.25 132) (end 189.5 129.75) (width 0.8) (layer F.Cu) (net 4))
+  (segment (start 165.75 132) (end 187.25 132) (width 0.8) (layer F.Cu) (net 4))
+  (segment (start 163.75 134) (end 165.75 132) (width 0.8) (layer F.Cu) (net 4))
+  (segment (start 163.75 136.25) (end 163.75 134) (width 0.8) (layer F.Cu) (net 4))
+  (segment (start 164 136.5) (end 163.75 136.25) (width 0.8) (layer F.Cu) (net 4))
+  (via (at 164 136.5) (size 1.7) (drill 0.8) (layers F.Cu B.Cu) (net 4))
+  (segment (start 164.592 137.092) (end 164 136.5) (width 0.8) (layer B.Cu) (net 4))
+  (segment (start 146.05 148.59) (end 149.59 148.59) (width 0.8) (layer B.Cu) (net 4))
+  (segment (start 151.368 150.368) (end 155.956 150.368) (width 0.8) (layer B.Cu) (net 4))
+  (segment (start 149.59 148.59) (end 151.368 150.368) (width 0.8) (layer B.Cu) (net 4))
+  (segment (start 163.068 150.368) (end 164.592 148.844) (width 0.8) (layer B.Cu) (net 4))
+  (segment (start 164.592 148.844) (end 164.592 142) (width 0.8) (layer B.Cu) (net 4))
+  (segment (start 164.592 142) (end 164.592 141.732) (width 0.8) (layer B.Cu) (net 4))
+  (segment (start 155.956 150.368) (end 163.068 150.368) (width 0.8) (layer B.Cu) (net 4))
+  (segment (start 164.75 132) (end 163.5 132) (width 0.8) (layer B.Cu) (net 5))
+  (segment (start 161.544 147.828) (end 162.56 146.812) (width 0.8) (layer B.Cu) (net 5))
+  (segment (start 157.422 147.828) (end 161.544 147.828) (width 0.8) (layer B.Cu) (net 5))
+  (segment (start 187.25 132) (end 189.5 129.75) (width 0.8) (layer B.Cu) (net 5))
+  (segment (start 189.5 129.75) (end 189.5 102.25) (width 0.8) (layer B.Cu) (net 5))
+  (segment (start 189.5 102.25) (end 187.25 100) (width 0.8) (layer B.Cu) (net 5))
+  (segment (start 187.25 100) (end 143 100) (width 0.8) (layer B.Cu) (net 5))
+  (segment (start 143 100) (end 141 102) (width 0.8) (layer B.Cu) (net 5))
+  (via (at 141 102) (size 1.7) (drill 0.8) (layers F.Cu B.Cu) (net 5))
+  (segment (start 141 102) (end 141.12 102.12) (width 0.8) (layer F.Cu) (net 5))
+  (segment (start 141.12 102.12) (end 141.12 105.16) (width 0.8) (layer F.Cu) (net 5))
+  (segment (start 164.75 132) (end 184 132) (width 0.8) (layer B.Cu) (net 5))
+  (segment (start 184 132) (end 187.25 132) (width 0.8) (layer B.Cu) (net 5))
+  (segment (start 162.56 139.81) (end 162.56 146.812) (width 0.8) (layer B.Cu) (net 5))
+  (segment (start 161.5 138.75) (end 162.56 139.81) (width 0.8) (layer B.Cu) (net 5))
+  (segment (start 161.5 134) (end 161.5 138.75) (width 0.8) (layer B.Cu) (net 5))
+  (segment (start 163.5 132) (end 161.5 134) (width 0.8) (layer B.Cu) (net 5))
+  (segment (start 154 147.828) (end 157.422 147.828) (width 0.8) (layer B.Cu) (net 5))
+  (segment (start 146.05 151.13) (end 148.62 151.13) (width 0.8) (layer B.Cu) (net 5))
+  (segment (start 152.578 147.828) (end 154 147.828) (width 0.8) (layer B.Cu) (net 5))
+  (segment (start 154 147.828) (end 155.956 147.828) (width 0.8) (layer B.Cu) (net 5))
+  (segment (start 152.25 147.5) (end 152.578 147.828) (width 0.8) (layer B.Cu) (net 5))
+  (via (at 152.25 147.5) (size 1.7) (drill 0.8) (layers F.Cu B.Cu) (net 5))
+  (segment (start 148.75 151) (end 152.25 147.5) (width 0.8) (layer F.Cu) (net 5))
+  (via (at 148.75 151) (size 1.7) (drill 0.8) (layers F.Cu B.Cu) (net 5))
+  (segment (start 148.62 151.13) (end 148.75 151) (width 0.8) (layer B.Cu) (net 5))
+  (segment (start 155.956 147.828) (end 157.422 147.828) (width 0.8) (layer B.Cu) (net 5))
   (segment (start 146.05 140.97) (end 148.082 140.97) (width 0.8) (layer B.Cu) (net 6))
   (segment (start 151.892 133.858) (end 156.21 129.54) (width 0.8) (layer B.Cu) (net 6))
