File: resources/hardware/head_board_wdriver/head_board.sch (KiCad schematic (older format))
At the start: 23 parts, among them IC1 ATMEGA328P-P, P1 SERIAL, P2 PI_CONN, P3 REED, P4 PR, P5 CAM_LEDS, P6 STEPPER, P7 PR_LED, P8 FDBK_LED, Q1 BC547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

Commit message: added stepper board
Parts:
- removed D2, D3: D, Diodes_ThroughHole:Diode_DO-41_SOD81_Horizontal_RM10, symbol D
- removed P1: SERIAL, Pin_Headers:Pin_Header_Straight_1x06, symbol CONN_01X06
- removed P6: STEPPER, Pin_Headers:Pin_Header_Straight_1x06, symbol CONN_01X06
- removed Q1, Q2: BC547, TO_SOT_Packages_THT:TO-92_Inline_Wide, symbol BC547
- removed R7, R8: 330 Ohm, Resistors_ThroughHole:Resistor_Horizontal_RM7mm, symbol R_Small
- added P1: SERIAL/RST, Pin_Headers:Pin_Header_Straight_1x03, symbol CONN_01X03
- added P6: STEPPER, Pin_Headers:Pin_Header_Straight_1x05, symbol CONN_01X05
- added U1: ULN2003, Housings_DIP:DIP-16_W7.62mm, symbol ULN2003
Connections:
- net labels removed: CTS, DTR, RX, TX, VCC
- wire segments 76 -> 58
- no-connect marks 38 -> 39
Other:
- moved on the sheet: P8, R6
